File: birdnet-mic-hat.kicad_sch (KiCad schematic)
At the start: 26 parts, among them J1 PJ-327A0-SMT, J3 DF40HC(3.5)-30DS-0.4V(51), Q1 MMBT3904, U1 TLV320ADC5140, U2 TPS7A2033PDBVR

Commit message: Apply 2026-10-18 design-review fixes before relayout
Schematic: R3 becomes a 100k SHDNZ pull-down; add 4.7k I2C pull-ups
(R9/R10), a 33R PDM_CLK series resistor (R11), and ESD9B5.0ST5G TVS
diodes on JACK_TIP/JACK_RING (D1/D2). C11 footprint unchanged (0603).

PCB: R11 at U1 pin 11, pull-ups and TVS diodes placed and routed;
direct top-copper ground bar from U1 AVSS (pin 4) to the VREF/MICBIAS/
AREG caps; C9 moved beside U2; U1 EPAD paste removed (vias to be
plugged at fab); ENIG finish; edge via moved inboard; new references
hidden.

Checkpoint only: C11 is parked off-board and its MIC_RING_N connection
is unrouted. This state precedes a full relayout.

Co-Authored-By: Claude Opus 5.5 <noreply@anthropic.com>
Parts:
- added D1, D2: ESD9B5.0ST5G, Diode_SMD:D_SOD-923, symbol Device:D_TVS
- added R10, R9: 4.7k, Resistor_SMD:R_0402_1005Metric, symbol Device:R
- added R11: 33, Resistor_SMD:R_0402_1005Metric, symbol Device:R
- R3: value 10k -> 100k
Connections:
- net GND: now also R3.1, D1.1 (A1), D2.1 (A1)
- net I2C_SCL: now also R9.2
- net I2C_SDA: now also R10.2
- net JACK_RING: now also D2.2 (A2)
- net JACK_TIP: now also D1.2 (A2)
- net PDM_CLK: now also R11.2; no longer U1.11 (IN3M_GPO3)
- net VCC_3V3: now also R10.1, R9.1; no longer R3.1
- new net: R11.1, U1.11 (IN3M_GPO3)
Other:
- note added: "R4/R5 hold the address straps low."
- note removed: "R4/R5 hold the address straps low. R3 pulls SHDNZ high; GPIO40 controls reset."
- moved on the sheet: R3

Commit message: Relayout: route board, swap J3 I2S/I2C GPIO assignment
Full re-route of the 2026-10-18 relayout. J3 signals were permuted so
I2S drops straight down from U1 pins 21-23: 8 SDOUT/GPIO42,
10 BCLK/GPIO41, 12 WS/GPIO40, 14 SCL/GPIO39, 16 SDA/GPIO38,
18 ADC_RST/GPIO47, 20 MIC_PRESENT/GPIO48. Firmware must follow.

U1 pad 4 zone connection set to solid (hard-wired AVSS bar).
DRC: 0 errors, 0 unconnected, parity 0; 2 known U1/J3 library
mismatch warnings. ERC: 0/0.

Co-Authored-By: Claude Opus 5.5 <noreply@anthropic.com>
Parts:
- added C13, C14: 10uF, Capacitor_SMD:C_0603_1608Metric, symbol Device:C
- added FB1: 600R@100MHz, Inductor_SMD:L_0402_1005Metric, symbol Device:FerriteBead
Connections:
- net ADC_RST: now also J3.18 (Pin_18); no longer J3.12 (Pin_12)
- net AVDD: now also C13.1, FB1.1; no longer C12.1, MK1.1 (VDD)
- net GND: now also C13.2, C14.2
- net I2C_SCL: now also J3.14 (Pin_14); no longer J3.8 (Pin_8)
- net I2C_SDA: now also J3.16 (Pin_16); no longer J3.10 (Pin_10)
- net I2S_BCLK: now also J3.10 (Pin_10); no longer J3.18 (Pin_18)
- net I2S_SDOUT: now also J3.8 (Pin_8); no longer J3.16 (Pin_16)
- net I2S_WS: now also J3.12 (Pin_12); no longer J3.14 (Pin_14)
- net VCC_3V3: now also C14.1
- new net MIC_VDD: C12.1, FB1.2, MK1.1 (VDD)
Other:
- note added: "10 BCLK / GPIO41"
- note added: "12 WS / GPIO40"
- note added: "14 SCL / GPIO39"
- note added: "16 SDA / GPIO38"
- note added: "18 ADC_RST / GPIO47"
- note added: "8 SDOUT / GPIO42"
- note removed: "10 SDA / GPIO41"
- note removed: "12 RESET / GPIO40"
- note removed: "14 WS / GPIO39"
- note removed: "16 SDOUT / GPIO38"
- note removed: "18 BCLK / GPIO47"
- note removed: "8 SCL / GPIO42"
